File: Preliminary_Schematic.kicad_sch (KiCad schematic)
At the start: 15 parts

Commit message: Footprints assigned to circuit components. Now layout generates without errors.
Parts:
- BT1: renamed from BT?; footprint (none) -> Battery:BatteryHolder_Keystone_2479_3xAAA
- D1, D2, D3, D4: renamed from D?; footprint (none) -> LED_SMD:LED_0201_0603Metric
- R1, R2, R3, R4, R5: renamed from R?; footprint (none) -> Resistor_SMD:R_0805_2012Metric_Pad1.20x1.40mm_HandSolder
- SW1, SW2, SW3, SW4: renamed from SW?; footprint (none) -> Button_Switch_SMD:SW_SPST_B3U-1000P
- gave numbers to parts that had none: 1
